File: circuit/Tortu/Tortu.kicad_pcb (KiCad board)
At the start: 2 copper layers, 94 x 81.9 mm, 21 parts

Commit message: v1.3
Parts:
- added Battery1: Battery, Connector_PinHeader_2.54mm:PinHeader_1x02_P2.54mm_Vertical, F.Cu at (165.1, 62.2)
- added SW1: SW_DPST_x2, Connector_PinHeader_2.54mm:PinHeader_1x02_P2.54mm_Vertical, F.Cu at (122.6, 73.0)
- R1: footprint Resistor_THT:R_Axial_DIN0204_L3.6mm_D1.6mm_P5.08mm_Horizontal -> Resistor_THT:R_Axial_DIN0207_L6.3mm_D2.5mm_P10.16mm_Horizontal
- moved C_Pico2 37.0 mm to (208.5, 132.1)
- moved C_Pico1 36.3 mm to (208.5, 128.3)
- moved SDCard1 35.9 mm to (200.7, 80.0), turned to -90 degrees
- moved MCU1 35.8 mm to (186.9, 114.3)
- moved Display1 32.0 mm to (165.1, 71.7), turned to 0 degrees
- moved C_Display1 26.3 mm to (160.0, 73.0), turned to 180 degrees
- moved C_SD1 21.0 mm to (186.7, 95.9), turned to -90 degrees
- moved C_Audio1 16.5 mm to (144.3, 82.8)
- moved AudioJack1 10.1 mm to (132.6, 124.0), turned to -90 degrees
- moved G*** 9.88 mm to (145.5, 106.7)
- moved C_Audio2 8.89 mm to (140.5, 82.8)
- moved R1 6.27 mm to (137.7, 113.8)
- moved LS1 3.81 mm to (122.7, 132.8), turned to 90 degrees
Connections:
- AudioAmp1 pad 5: GPIO2 -> GPIO6
- AudioAmp1 pad 6: GPIO0 -> GPIO4
- AudioAmp1 pad 7: GPIO1 -> GPIO5
- LX-LCBST1 pad 1: unconnected-(LX-LCBST1-B+-Pad1) -> Net-(Battery1-Pin_1)
- LX-LCBST1 pad 2: unconnected-(LX-LCBST1-B--Pad2) -> Net-(Battery1-Pin_2)
- LX-LCBST1 pad 3: Vin -> Net-(LX-LCBST1-V0+)
- MCU1 pad 6: unconnected-(MCU1-GPIO4-Pad6) -> GPIO4
- MCU1 pad 7: unconnected-(MCU1-GPIO5-Pad7) -> GPIO5
- MCU1 pad 9: unconnected-(MCU1-GPIO6-Pad9)_1 -> GPIO6
- RV1 pad 2: Net-(LS1-Pad1) -> Net-(AudioAmp1-OUTP)
- RV1 pad 3: Net-(AudioAmp1-OUTP) -> Net-(LS1-Pad1)
Routing:
- net GPIO6: track 0.00 -> 152.4 mm
- net GPIO5: track 0.00 -> 139.5 mm
- net GPIO4: track 0.00 -> 138.7 mm
- net GPIO1: track 125.0 -> 0.00 mm
- net GPIO0: track 86.2 -> 0.00 mm
- net GPIO2: track 77.5 -> 0.00 mm
- net GPIO10: track 106.7 -> 30.9 mm
- net GPIO17: track 13.5 -> 84.7 mm
- net GPIO11: track 101.1 -> 30.8 mm
- net GPIO12: track 95.5 -> 29.7 mm
- net Vin: track 97.3 -> 160.6 mm
- net GPIO21: track 25.7 -> 87.2 mm
- net GPIO20: track 31.9 -> 90.0 mm
- net Net-(Battery1-Pin_2): track 0.00 -> 53.8 mm
- net GPIO13: track 101.4 -> 51.5 mm, vias 1 -> 0
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Other:
- board text added: "2025-01-02 v1.3"
- board text removed: "2024-10-19 v1.1"
