File: circuit/Tortu/Tortu.kicad_sch (KiCad schematic)
At the start: 20 parts

Commit message: v1.3
Parts:
- added Battery1: Battery, Connector_PinHeader_2.54mm:PinHeader_1x02_P2.54mm_Vertical, symbol Connector:Conn_01x02_Pin
- added SW1: SW_DPST_x2, Connector_PinHeader_2.54mm:PinHeader_1x02_P2.54mm_Vertical, symbol Switch:SW_DPST_x2
- R1: footprint Resistor_THT:R_Axial_DIN0204_L3.6mm_D1.6mm_P5.08mm_Horizontal -> Resistor_THT:R_Axial_DIN0207_L6.3mm_D2.5mm_P10.16mm_Horizontal
Connections:
- net Vin: now also SW1.2 (B); no longer LX-LCBST1.3 (V0+)
- net at LS1.1, R1.1: now also RV1.3; no longer RV1.2
- net at LX-LCBST1.1 (B+): now also Battery1.1 (Pin_1)
- net at LX-LCBST1.2 (B-): now also Battery1.2 (Pin_2)
- net at AudioAmp1.8 (OUTP): now also RV1.2; no longer RV1.3
- net GPIO4: now reaches MCU1.6 (GPIO4)
- net GPIO4: now also AudioAmp1.6 (BCLK)
- net GPIO5: now reaches MCU1.7 (GPIO5)
- net GPIO5: now also AudioAmp1.7 (LRC)
- net GPIO6: now reaches MCU1.9 (GPIO6)
- net GPIO6: now also AudioAmp1.5 (DIN)
- net GPIO0: no longer names the net of MCU1.1 (GPIO0)
- net GPIO0: no longer AudioAmp1.6 (BCLK)
- net GPIO1: no longer names the net of MCU1.2 (GPIO1)
- net GPIO1: no longer AudioAmp1.7 (LRC)
- net GPIO2: no longer names the net of MCU1.4 (GPIO2)
- net GPIO2: no longer AudioAmp1.5 (DIN)
- new net: LX-LCBST1.3 (V0+), SW1.1 (A)
- no-connect marks 23 -> 21
Other:
- moved on the sheet: LX-LCBST1, RV1
